Commit message: Added conditional blocks to allow for a variable number of wegs per wheel to be stored in the xacro file.

File: adabot_description/urdf/adabot.main.xacro (robot description, xacro)
@@ -4,33 +4,31 @@
          Properties for the robot bodies
     -->
-    <xacro:property name="PI" value="3.1415926535897931 "/>
-    <xacro:property name="SCALE" value="2" />
+    <xacro:property name="PI" value="3.1415926535897931"/>
     <!-- Typical density of plastics -->
     <xacro:property name="mat_density" value="1000.0" />
-    <!-- Chassis parameters -->
-    <xacro:property name="ch_density_factor" value="0.4" />
-    <xacro:property name="ch_density" value="${mat_density * ch_density_factor}" />
-    <xacro:property name="ch_length"  value="${0.100 * SCALE}" />
-    <xacro:property name="ch_width"   value="${0.070 * SCALE}" />
-    <xacro:property name="ch_height"  value="${0.035 * SCALE}" />
-    <xacro:property name="ch_mass"    value="${ch_density * ch_length * ch_width * ch_height}" />
     <!-- Wheel parameters -->
-    <xacro:property name="wh_density_factor" value="0.4" />
-    <xacro:property name="wh_density" value="${mat_density * wh_density_factor}" />
-    <xacro:property name="wh_radius"  value="${0.020 * SCALE}" />
-    <xacro:property name="wh_length"  value="${0.005 * SCALE}" />
-    <xacro:property name="wh_mass"    value="${wh_density * PI * (wh_radius**2) * wh_length}" />
-    <!-- Weg parameters -->
-    <xacro:property name="wg_length" value="${wh_radius*2}" />
-    <xacro:property name="wg_width"  value="${0.001 * SCALE}" />
-    <xacro:property name="wg_height" value="${0.002 * SCALE}" />
-    <xacro:property name="wg_mass"   value="${mat_density * wg_length * wg_width * wg_height}" />
+    <xacro:property name="wh_radius" value="0.02" />
+    <xacro:property name="wh_length" value="0.005" />
+    <xacro:property name="wh_mass" value="${mat_density*PI*(wh_radius**2)*wh_length}" />
     <!-- Axle parameters -->
     <xacro:property name="ax_axis" value="0 1 0" />
+    <!-- Chassis parameters -->
+    <xacro:property name="ch_length" value="0.1" />
+    <xacro:property name="ch_width" value="0.07" />
+    <xacro:property name="ch_height" value="0.035" />
+    <xacro:property name="ch_mass" value="${mat_density*ch_length*ch_width*ch_height}" />
+    <!-- Weg parameters -->
+    <xacro:property name="wg_per_wheel" value="2" />
+    <xacro:property name="wg_length" value="${wh_radius*2}" />
+    <xacro:property name="wg_width" value="0.001" />
+    <xacro:property name="wg_height" value="0.002" />
+    <xacro:property name="wg_mass" value="${mat_density*wg_length*wg_width*wg_height}" />
     <!-- Vertical offset so that the robot starts above ground -->
-    <xacro:property name="zoffset" value="${wh_radius*1.1/2 * 10}" />
+    <xacro:property name="zoffset" value="${wh_radius*1.1/2}" />
     <!--
          Properties for names, colors, and Gazebo
     -->
+    <!-- The chassis is the parent of several other links, so we need it's name -->
+    <xacro:property name="chassisname" value="base_link" />
     <!-- Import colors defined for Rviz -->
     <xacro:include filename="$(find adabot_description)/urdf/adabot.materials.xacro" />
@@ -54,5 +52,5 @@
     -->
     <xacro:macro name="weg" params="wheel number parent total">
-        <xacro:property name="wg_name" value="wg_${wheel}_${number}" />
+        <xacro:property name="wg_name" value="wg-${wheel}-${number}" />
         <link name="${wg_name}">
             <visual>
@@ -75,5 +73,5 @@
             </inertial>
         </link>
-        <joint name="${wg_name}_joint" type="prismatic">
+        <joint name="${wg_name}-joint" type="prismatic">
             <parent link="${parent}" />
             <child link="${wg_name}" />
@@ -85,5 +83,5 @@
          Macro for creating wheel geoms
     -->
-    <xacro:property name="wh_origin_geom">
+    <xacro:property name="wh_orig_geom">
         <!-- Cylinders default with their height along the z axis -->
         <origin rpy="1.57075 0 0" xyz="0 0 0" />
@@ -100,17 +98,15 @@
     -->
     <xacro:macro name="wheel" params="reflect_lr reflect_fb suffix parent">
-        <xacro:property name="wh_name" value="wh_${suffix}" />
-        <xacro:gz_wheel_material name="${wh_name}" />
+        <xacro:property name="wh_name" value="wh-${suffix}" />
         <link name="${wh_name}">
             <visual>
-                <xacro:insert_block name="wh_origin_geom" />
+                <xacro:insert_block name="wh_orig_geom" />
                 <material name="black" />
             </visual>
             <collision>
-                <xacro:insert_block name="wh_origin_geom" />
+                <xacro:insert_block name="wh_orig_geom" />
             </collision>
             <inertial>
                 <mass value="${wh_mass}" />
-                <origin rpy="1.57075 0 0" xyz="0 0 0" />
                 <inertia
                     ixx="${(1/12)*wh_mass*(3*wh_radius**2 + wh_length**2)}"
@@ -123,9 +119,8 @@
             </inertial>
         </link>
-        <joint name="ax_${suffix}" type="continuous">
+        <joint name="ax-${suffix}" type="continuous">
             <parent link="${parent}" />
             <child link="${wh_name}" />
-            <!-- <origin rpy="0 0 0" xyz="${ch_length/2*reflect_fb} ${(wh_length+ch_width)/2*reflect_lr} ${zoffset}" /> -->
-            <origin rpy="0 0 0" xyz="${ch_length/2*reflect_fb} ${(wh_length+ch_width)/2*reflect_lr} 0" />
+            <origin rpy="0 0 0" xyz="${ch_length/2*reflect_fb} ${(wh_length+ch_width)/2*reflect_lr} ${zoffset}" />
             <axis xyz="${ax_axis}" />
         </joint>
@@ -137,16 +132,34 @@
                 (5) have some ugly conditionals below
         -->
-        <xacro:weg wheel="${suffix}" number="1" parent="${wh_name}" total="5" />
-        <xacro:weg wheel="${suffix}" number="2" parent="${wh_name}" total="5" />
-        <xacro:weg wheel="${suffix}" number="3" parent="${wh_name}" total="5" />
-        <xacro:weg wheel="${suffix}" number="4" parent="${wh_name}" total="5" />
-        <xacro:weg wheel="${suffix}" number="5" parent="${wh_name}" total="5" />
+        <xacro:if value="${wg_per_wheel > 0}">
+            <xacro:weg wheel="${suffix}" number="1" parent="${wh_name}" total="${wg_per_wheel}" />
+        </xacro:if>
+        <xacro:if value="${wg_per_wheel > 1}">
+            <xacro:weg wheel="${suffix}" number="2" parent="${wh_name}" total="${wg_per_wheel}" />
+        </xacro:if>
+        <xacro:if value="${wg_per_wheel > 2}">
+            <xacro:weg wheel="${suffix}" number="3" parent="${wh_name}" total="${wg_per_wheel}" />
+        </xacro:if>
+        <xacro:if value="${wg_per_wheel > 3}">
+            <xacro:weg wheel="${suffix}" number="4" parent="${wh_name}" total="${wg_per_wheel}" />
+        </xacro:if>
+        <xacro:if value="${wg_per_wheel > 4}">
+            <xacro:weg wheel="${suffix}" number="5" parent="${wh_name}" total="${wg_per_wheel}" />
+        </xacro:if>
+        <xacro:if value="${wg_per_wheel > 5}">
+            <xacro:weg wheel="${suffix}" number="6" parent="${wh_name}" total="${wg_per_wheel}" />
+        </xacro:if>
+        <xacro:if value="${wg_per_wheel > 6}">
+            <xacro:weg wheel="${suffix}" number="7" parent="${wh_name}" total="${wg_per_wheel}" />
+        </xacro:if>
+        <xacro:if value="${wg_per_wheel > 7}">
+            <xacro:weg wheel="${suffix}" number="8" parent="${wh_name}" total="${wg_per_wheel}" />
+        </xacro:if>
     </xacro:macro>
     <!--
          Macro for creating the chassis' geom
     -->
-    <xacro:property name="ch_origin_geom">
-        <!-- <origin rpy="0 0 0" xyz="0 0 ${zoffset}" /> -->
-        <origin rpy="0 0 0" xyz="0 0 0" />
+    <xacro:property name="ch_orig_geom">
+        <origin rpy="0 0 0" xyz="0 0 ${zoffset}" />
         <geometry>
             <box size="${ch_length} ${ch_width} ${ch_height}" />
@@ -155,20 +168,15 @@
     <!--
          The main chassis/body
-            Note: the chassis is connect to the world link so that it's link frame is
-            easier to visualize. This will also help when we start to include multiple
-            robots.
     -->
-    <link name="world" />
-    <link name="chassis">
+    <link name="${chassisname}">
         <visual>
-            <xacro:insert_block name="ch_origin_geom" />
+            <xacro:insert_block name="ch_orig_geom" />
             <material name="white" />
         </visual>
         <collision>
-            <xacro:insert_block name="ch_origin_geom" />
+            <xacro:insert_block name="ch_orig_geom" />
         </collision>
         <inertial>
             <mass value="${ch_mass}" />
-            <!-- <origin xyz="0 0 ${zoffset}" rpy="0 0 0"/> -->
             <inertia
                 ixx="${(1/12)*ch_mass*(ch_width**2 + ch_height**2)}"
@@ -181,32 +189,10 @@
         </inertial>
     </link>
-    <joint name="world_joint" type="floating">
-        <!-- <origin xyz="0 0 0" rpy="0 0 0" /> -->
-        <origin xyz="0 0 ${zoffset}" rpy="0 0 0" />
-        <parent link="world" />
-        <child link="chassis" />
-    </joint>
     <!--
          Macro calls for creating wheels
     -->
-    <xacro:wheel reflect_lr="-1" reflect_fb="1"  suffix="front_left"  parent="chassis" />
-    <xacro:wheel reflect_lr="1"  reflect_fb="1"  suffix="front_right" parent="chassis" />
-    <xacro:wheel reflect_lr="-1" reflect_fb="-1" suffix="back_left"   parent="chassis" />
-    <xacro:wheel reflect_lr="1"  reflect_fb="-1" suffix="back_right"  parent="chassis" />
-    <!--
-         Add a transmission for ros_control so that it can control the wheel motors
-    -->
-    <transmission name="tran_front_left" type="SimpleTransmission">
-        <type>transmission_interface/SimpleTransmission</type>
-        <joint name="ax_front_left">
-            <hardwareInterface>hardware_interface/EffortJointInterface</hardwareInterface>
-        </joint>
-        <actuator name="motor_front_left">
-            <hardwareInterface>hardware_interface/EffortJointInterface</hardwareInterface>
-            <mechanicalReduction>1</mechanicalReduction>
-        </actuator>
-    </transmission>
-    <!--
-         Add a Gazebo world element as a reference
-    -->
+    <xacro:wheel reflect_lr="-1" reflect_fb="1" suffix="front-left" parent="${chassisname}" />
+    <xacro:wheel reflect_lr="1" reflect_fb="1" suffix="front-right" parent="${chassisname}" />
+    <xacro:wheel reflect_lr="-1" reflect_fb="-1" suffix="back-left" parent="${chassisname}" />
+    <xacro:wheel reflect_lr="1" reflect_fb="-1" suffix="back-right" parent="${chassisname}" />
 </robot>

Commit message: Updated file to match 'Master'

File: adabot_description/urdf/adabot.main.xacro (robot description, xacro)
@@ -4,31 +4,34 @@
          Properties for the robot bodies
     -->
-    <xacro:property name="PI" value="3.1415926535897931"/>
+    <xacro:property name="PI" value="3.1415926535897931 "/>
+    <xacro:property name="SCALE" value="2" />
     <!-- Typical density of plastics -->
     <xacro:property name="mat_density" value="1000.0" />
+    <!-- Chassis parameters -->
+    <xacro:property name="ch_density_factor" value="0.4" />
+    <xacro:property name="ch_density" value="${mat_density * ch_density_factor}" />
+    <xacro:property name="ch_length"  value="${0.100 * SCALE}" />
+    <xacro:property name="ch_width"   value="${0.070 * SCALE}" />
+    <xacro:property name="ch_height"  value="${0.035 * SCALE}" />
+    <xacro:property name="ch_mass"    value="${ch_density * ch_length * ch_width * ch_height}" />
     <!-- Wheel parameters -->
-    <xacro:property name="wh_radius" value="0.02" />
-    <xacro:property name="wh_length" value="0.005" />
-    <xacro:property name="wh_mass" value="${mat_density*PI*(wh_radius**2)*wh_length}" />
-    <!-- Axle parameters -->
-    <xacro:property name="ax_axis" value="0 1 0" />
-    <!-- Chassis parameters -->
-    <xacro:property name="ch_length" value="0.1" />
-    <xacro:property name="ch_width" value="0.07" />
-    <xacro:property name="ch_height" value="0.035" />
-    <xacro:property name="ch_mass" value="${mat_density*ch_length*ch_width*ch_height}" />
+    <xacro:property name="wh_density_factor" value="0.4" />
+    <xacro:property name="wh_density" value="${mat_density * wh_density_factor}" />
+    <xacro:property name="wh_radius"  value="${0.020 * SCALE}" />
+    <xacro:property name="wh_length"  value="${0.005 * SCALE}" />
+    <xacro:property name="wh_mass"    value="${wh_density * PI * (wh_radius**2) * wh_length}" />
     <!-- Weg parameters -->
     <xacro:property name="wg_per_wheel" value="2" />
     <xacro:property name="wg_length" value="${wh_radius*2}" />
-    <xacro:property name="wg_width" value="0.001" />
-    <xacro:property name="wg_height" value="0.002" />
-    <xacro:property name="wg_mass" value="${mat_density*wg_length*wg_width*wg_height}" />
+    <xacro:property name="wg_width"  value="${0.001 * SCALE}" />
+    <xacro:property name="wg_height" value="${0.002 * SCALE}" />
+    <xacro:property name="wg_mass"   value="${mat_density * wg_length * wg_width * wg_height}" />
+    <!-- Axle parameters -->
+    <xacro:property name="ax_axis" value="0 1 0" />
     <!-- Vertical offset so that the robot starts above ground -->
-    <xacro:property name="zoffset" value="${wh_radius*1.1/2}" />
+    <xacro:property name="zoffset" value="${wh_radius*1.1/2 * 10}" />
     <!--
          Properties for names, colors, and Gazebo
     -->
-    <!-- The chassis is the parent of several other links, so we need it's name -->
-    <xacro:property name="chassisname" value="base_link" />
     <!-- Import colors defined for Rviz -->
     <xacro:include filename="$(find adabot_description)/urdf/adabot.materials.xacro" />
@@ -52,5 +55,5 @@
     -->
     <xacro:macro name="weg" params="wheel number parent total">
-        <xacro:property name="wg_name" value="wg-${wheel}-${number}" />
+        <xacro:property name="wg_name" value="wg_${wheel}_${number}" />
         <link name="${wg_name}">
             <visual>
@@ -73,5 +76,5 @@
             </inertial>
         </link>
-        <joint name="${wg_name}-joint" type="prismatic">
+        <joint name="${wg_name}_joint" type="prismatic">
             <parent link="${parent}" />
             <child link="${wg_name}" />
@@ -83,5 +86,5 @@
          Macro for creating wheel geoms
     -->
-    <xacro:property name="wh_orig_geom">
+    <xacro:property name="wh_origin_geom">
         <!-- Cylinders default with their height along the z axis -->
         <origin rpy="1.57075 0 0" xyz="0 0 0" />
@@ -98,15 +101,17 @@
     -->
     <xacro:macro name="wheel" params="reflect_lr reflect_fb suffix parent">
-        <xacro:property name="wh_name" value="wh-${suffix}" />
+        <xacro:property name="wh_name" value="wh_${suffix}" />
+        <xacro:gz_wheel_material name="${wh_name}" />
         <link name="${wh_name}">
             <visual>
-                <xacro:insert_block name="wh_orig_geom" />
+                <xacro:insert_block name="wh_origin_geom" />
                 <material name="black" />
             </visual>
             <collision>
-                <xacro:insert_block name="wh_orig_geom" />
+                <xacro:insert_block name="wh_origin_geom" />
             </collision>
             <inertial>
                 <mass value="${wh_mass}" />
+                <origin rpy="1.57075 0 0" xyz="0 0 0" />
                 <inertia
                     ixx="${(1/12)*wh_mass*(3*wh_radius**2 + wh_length**2)}"
@@ -119,8 +124,9 @@
             </inertial>
         </link>
-        <joint name="ax-${suffix}" type="continuous">
+        <joint name="ax_${suffix}" type="continuous">
             <parent link="${parent}" />
             <child link="${wh_name}" />
-            <origin rpy="0 0 0" xyz="${ch_length/2*reflect_fb} ${(wh_length+ch_width)/2*reflect_lr} ${zoffset}" />
+            <!-- <origin rpy="0 0 0" xyz="${ch_length/2*reflect_fb} ${(wh_length+ch_width)/2*reflect_lr} ${zoffset}" /> -->
+            <origin rpy="0 0 0" xyz="${ch_length/2*reflect_fb} ${(wh_length+ch_width)/2*reflect_lr} 0" />
             <axis xyz="${ax_axis}" />
         </joint>
@@ -160,6 +166,7 @@
          Macro for creating the chassis' geom
     -->
-    <xacro:property name="ch_orig_geom">
-        <origin rpy="0 0 0" xyz="0 0 ${zoffset}" />
+    <xacro:property name="ch_origin_geom">
+        <!-- <origin rpy="0 0 0" xyz="0 0 ${zoffset}" /> -->
+        <origin rpy="0 0 0" xyz="0 0 0" />
         <geometry>
             <box size="${ch_length} ${ch_width} ${ch_height}" />
@@ -168,15 +175,20 @@
     <!--
          The main chassis/body
-    -->
-    <link name="${chassisname}">
+            Note: the chassis is connect to the world link so that it's link frame is
+            easier to visualize. This will also help when we start to include multiple
+            robots.
+    -->
+    <link name="world" />
+    <link name="chassis">
         <visual>
-            <xacro:insert_block name="ch_orig_geom" />
+            <xacro:insert_block name="ch_origin_geom" />
             <material name="white" />
         </visual>
         <collision>
-            <xacro:insert_block name="ch_orig_geom" />
+            <xacro:insert_block name="ch_origin_geom" />
         </collision>
         <inertial>
             <mass value="${ch_mass}" />
+            <!-- <origin xyz="0 0 ${zoffset}" rpy="0 0 0"/> -->
             <inertia
                 ixx="${(1/12)*ch_mass*(ch_width**2 + ch_height**2)}"
@@ -189,10 +201,32 @@
         </inertial>
     </link>
+    <joint name="world_joint" type="floating">
+        <!-- <origin xyz="0 0 0" rpy="0 0 0" /> -->
+        <origin xyz="0 0 ${zoffset}" rpy="0 0 0" />
+        <parent link="world" />
+        <child link="chassis" />
+    </joint>
     <!--
          Macro calls for creating wheels
     -->
-    <xacro:wheel reflect_lr="-1" reflect_fb="1" suffix="front-left" parent="${chassisname}" />
-    <xacro:wheel reflect_lr="1" reflect_fb="1" suffix="front-right" parent="${chassisname}" />
-    <xacro:wheel reflect_lr="-1" reflect_fb="-1" suffix="back-left" parent="${chassisname}" />
-    <xacro:wheel reflect_lr="1" reflect_fb="-1" suffix="back-right" parent="${chassisname}" />
+    <xacro:wheel reflect_lr="-1" reflect_fb="1"  suffix="front_left"  parent="chassis" />
+    <xacro:wheel reflect_lr="1"  reflect_fb="1"  suffix="front_right" parent="chassis" />
+    <xacro:wheel reflect_lr="-1" reflect_fb="-1" suffix="back_left"   parent="chassis" />
+    <xacro:wheel reflect_lr="1"  reflect_fb="-1" suffix="back_right"  parent="chassis" />
+    <!--
+         Add a transmission for ros_control so that it can control the wheel motors
+    -->
+    <transmission name="tran_front_left" type="SimpleTransmission">
+        <type>transmission_interface/SimpleTransmission</type>
+        <joint name="ax_front_left">
+            <hardwareInterface>hardware_interface/EffortJointInterface</hardwareInterface>
+        </joint>
+        <actuator name="motor_front_left">
+            <hardwareInterface>hardware_interface/EffortJointInterface</hardwareInterface>
+            <mechanicalReduction>1</mechanicalReduction>
+        </actuator>
+    </transmission>
+    <!--
+         Add a Gazebo world element as a reference
+    -->
 </robot>

Commit message: Added terminal input parameters to the launch file

File: adabot_description/urdf/adabot.main.xacro (robot description, xacro)
@@ -11,6 +11,6 @@
     <xacro:property name="ch_density_factor" value="0.4" />
     <xacro:property name="ch_density" value="${mat_density * ch_density_factor}" />
-    <xacro:property name="ch_length"  value="${0.100 * SCALE}" />
-    <xacro:property name="ch_width"   value="${0.070 * SCALE}" />
+    <xacro:property name="ch_length"  value="${$(arg ch_length) * SCALE}" />
+    <xacro:property name="ch_width"   value="${$(arg ch_width) * SCALE}" />
     <xacro:property name="ch_height"  value="${0.035 * SCALE}" />
     <xacro:property name="ch_mass"    value="${ch_density * ch_length * ch_width * ch_height}" />
@@ -18,13 +18,13 @@
     <xacro:property name="wh_density_factor" value="0.4" />
     <xacro:property name="wh_density" value="${mat_density * wh_density_factor}" />
-    <xacro:property name="wh_radius"  value="${0.020 * SCALE}" />
+    <xacro:property name="wh_radius"  value="${$(arg wh_radius) * SCALE}" />
     <xacro:property name="wh_length"  value="${0.005 * SCALE}" />
     <xacro:property name="wh_mass"    value="${wh_density * PI * (wh_radius**2) * wh_length}" />
     <!-- Weg parameters -->
-    <xacro:property name="wg_per_wheel" value="2" />
-    <xacro:property name="wg_length" value="${wh_radius*2}" />
-    <xacro:property name="wg_width"  value="${0.001 * SCALE}" />
-    <xacro:property name="wg_height" value="${0.002 * SCALE}" />
-    <xacro:property name="wg_mass"   value="${mat_density * wg_length * wg_width * wg_height}" />
+    <xacro:property name="wg_per_wheel" value="$(arg wg_per_wheel)" />
+    <xacro:property name="wg_length"    value="${wh_radius*2}" />
+    <xacro:property name="wg_width"     value="${0.001 * SCALE}" />
+    <xacro:property name="wg_height"    value="${0.002 * SCALE}" />
+    <xacro:property name="wg_mass"      value="${mat_density * wg_length * wg_width * wg_height}" />
     <!-- Axle parameters -->
     <xacro:property name="ax_axis" value="0 1 0" />
@@ -162,4 +162,7 @@
             <xacro:weg wheel="${suffix}" number="8" parent="${wh_name}" total="${wg_per_wheel}" />
         </xacro:if>
+        <xacro:if value="${wg_per_wheel > 8}">
+            <xacro:weg wheel="${suffix}" number="9" parent="${wh_name}" total="${wg_per_wheel}" />
+        </xacro:if>
     </xacro:macro>
     <!--
